Commit message: New chasis

File: urdf/macros.xacro (robot description, xacro)
@@ -110,3 +110,30 @@
   </transmission>
 </xacro:macro>
+<xacro:macro name="top_cover_two_cameras_macro" params="parent_link">
+  <link name="top_cover_two_cameras_link">
+    <inertial>
+      <origin xyz="0 0 0" rpy="0 0 0" />
+      <mass value="0.5" /> <!-- Ajusta la masa según corresponda -->
+      <inertia ixx="0.001" ixy="0" ixz="0" iyy="0.001" iyz="0" izz="0.001" />
+    </inertial>
+    <visual>
+      <origin xyz="0 0 0" rpy="0 0 0" />
+      <geometry>
+        <mesh filename="package://deepracer_simulation/meshes/top_cover_two_cameras.STL" scale="1 1 1" />
+      </geometry>
+      <material name="blue" /> <!-- Usa un material existente -->
+    </visual>
+    <collision>
+      <origin xyz="0 0 0" rpy="0 0 0" />
+      <geometry>
+        <mesh filename="package://deepracer_simulation/meshes/top_cover_two_cameras.STL" scale="1 1 1" />
+      </geometry>
+    </collision>
+  </link>
+  <joint name="top_cover_two_cameras_joint" type="fixed">
+    <origin xyz="0.03 0 -0.01" rpy="-1.57 3.14 0" /> <!-- Ajusta posición relativa -->
+    <parent link="${parent_link}" />
+    <child link="top_cover_two_cameras_link" />
+  </joint>
+</xacro:macro>
 </robot>

File: urdf/racecar.xacro (robot description, xacro)
@@ -7,5 +7,5 @@
     <visual>
       <xacro:chassis_geometry/>
-      <material name="blue" />
+      <material name="green" />
     </visual>
   </link>
@@ -25,4 +25,5 @@
     <child link="chassis_inertia" />
   </joint>
+  <xacro:top_cover_two_cameras_macro parent_link="chassis" />
   <!-- Add the left rear wheel with its joints and tranmissions -->
   <link name="left_rear_wheel">
@@ -155,5 +156,5 @@
       <origin xyz="0 0 0" rpy="0 0 0"/>
       <geometry>
-        <box size="0.033 0.175 0.030"/>
+        <box size="0.033 0.1 0.030"/> <!-- Tamaño caja representacion camara -->
       </geometry>
     </collision>
@@ -161,5 +162,5 @@
       <origin xyz="0 0 0" rpy="0 0 0"/>
       <geometry>
-        <box size="0.033 0.175 0.030"/>
+        <box size="0.033 0.1 0.030"/> <!-- Tamaño caja representacion camara -->
       </geometry>
       <material name="red"/>
