Commit message: Update racecar.xacro

File: urdf/racecar.xacro (robot description, xacro)
@@ -156,5 +156,5 @@
       <origin xyz="0 0 0" rpy="0 0 0"/>
       <geometry>
-        <box size="0.033 0.1 0.030"/> <!-- Tamaño caja representacion camara -->
+        <box size="0.033 0.030 0.030"/> <!-- Tamaño caja representacion camara -->
       </geometry>
     </collision>
@@ -162,5 +162,5 @@
       <origin xyz="0 0 0" rpy="0 0 0"/>
       <geometry>
-        <box size="0.033 0.1 0.030"/> <!-- Tamaño caja representacion camara -->
+        <box size="0.033 0.030 0.030"/> <!-- Tamaño caja representacion camara -->
       </geometry>
       <material name="red"/>
@@ -168,5 +168,5 @@
   </link>
   <joint name="zed_camera_joint" type="fixed">
-    <origin xyz="0.20 0 0.10" rpy="0 0.2731415 0"/>
+    <origin xyz="0.25 0 0.10" rpy="0 0.2731415 0"/> <!-- Cambiar posición y angulación de la cámara -->
     <parent link="chassis"/>
     <child link="zed_camera_link"/>
